File: Board/Board.brd (EAGLE design)
At the start: 72 x 50 mm, 24 parts, among them IC1 LM334, T1 BC807

Commit message: increased constant current feedback resistor
Parts:
- R2: value 3R3 -> 36
Changed lines of the file:
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@@
 <drawing>
 <settings>
-<setting alwaysvectorfont="yes"/>
+<setting alwaysvectorfont="no"/>
 <setting verticaltext="up"/>
 </settings>
@@
 </layers>
 <board>
-<fusionsync huburn="a.cGVyc29uYWw6dWUyOWFjMzc0" projecturn="a.cGVyc29uYWw6dWUyOWFjMzc0IzIwMTgxMTA5MTU5MzcxODUx" f3durn="urn:adsk.wipprod:dm.lineage:8R8TAl3XTbGenGFVYcsrqQ" pcbguid="c32a4f4f-8cd4-4b95-b40a-19347d32ef6f" lastpulledtime="2018-11-11T17:12:34Z" lastsyncedchangeguid="f148739b-0e27-b40c-a1d0-ee1bb420b8f3"/>
+<fusionsync huburn="a.cGVyc29uYWw6dWUyOWFjMzc0" projecturn="a.cGVyc29uYWw6dWUyOWFjMzc0IzIwMTgxMTA5MTU5MzcxODUx" f3durn="urn:adsk.wipprod:dm.lineage:8R8TAl3XTbGenGFVYcsrqQ" pcbguid="c32a4f4f-8cd4-4b95-b40a-19347d32ef6f" lastpulledtime="2018-12-01T15:07:32Z" lastsyncedchangeguid="c96938d0-b081-732c-ddc0-3cabcccae12e"/>
 <plain>
 <text x="11.5" y="40.5" size="2.5" layer="21" font="fixed" align="center">+</text>
@@
 https://www.conrad.de/de/tru-components-tc-2024-sw203-universal-gehaeuse-72-x-50-x-26-abs-schwarz-1-st-1588559.html</text>
 <text x="52" y="2" size="1.016" layer="22" rot="MR0" align="center">https://github.com/dangrie158/AdapterBox</text>
-<hole x="3" y="3" drill="3"/>
-<hole x="69" y="3" drill="3"/>
-<hole x="69" y="47" drill="3"/>
-<hole x="3" y="47" drill="3"/>
-<wire x1="3" y1="0" x2="69" y2="0" width="0.254" layer="20"/>
-<wire x1="69" y1="0" x2="72" y2="3" width="0.254" layer="20" curve="90"/>
-<wire x1="72" y1="3" x2="72" y2="47" width="0.254" layer="20"/>
-<wire x1="72" y1="47" x2="69" y2="50" width="0.254" layer="20" curve="90"/>
-<wire x1="69" y1="50" x2="3" y2="50" width="0.254" layer="20"/>
-<wire x1="3" y1="50" x2="0" y2="47" width="0.254" layer="20" curve="90"/>
-<wire x1="0" y1="47" x2="0" y2="3" width="0.254" layer="20"/>
-<wire x1="0" y1="3" x2="3" y2="0" width="0.254" layer="20" curve="90"/>
 <text x="19.825" y="34" size="1.27" layer="25" align="center-left">ON</text>
 <text x="44" y="5" size="6.4516" layer="21" font="vector" align="center">-</text>
@@
 <rectangle x1="62.8735" y1="7.8515" x2="63.6935" y2="7.8925" layer="22" rot="R180"/>
 <rectangle x1="62.9145" y1="7.8925" x2="63.6525" y2="7.9335" layer="22" rot="R180"/>
+<hole x="3" y="3" drill="3"/>
+<hole x="69" y="3" drill="3"/>
+<hole x="69" y="47" drill="3"/>
+<hole x="3" y="47" drill="3"/>
+<wire x1="3" y1="0" x2="69" y2="0" width="0.254" layer="20"/>
+<wire x1="69" y1="0" x2="72" y2="3" width="0.254" layer="20" curve="90"/>
+<wire x1="72" y1="3" x2="72" y2="47" width="0.254" layer="20"/>
+<wire x1="72" y1="47" x2="69" y2="50" width="0.254" layer="20" curve="90"/>
+<wire x1="69" y1="50" x2="3" y2="50" width="0.254" layer="20"/>
+<wire x1="3" y1="50" x2="0" y2="47" width="0.254" layer="20" curve="90"/>
+<wire x1="0" y1="47" x2="0" y2="3" width="0.254" layer="20"/>
+<wire x1="0" y1="3" x2="3" y2="0" width="0.254" layer="20" curve="90"/>
 </plain>
 <attributes>
@@
 <attribute name="VALUE" x="29.499996875" y="38.6354" size="0.8128" layer="26" rot="MR180" align="top-center"/>
 </element>
-<element name="R2" library="rcl" library_urn="urn:adsk.eagle:library:334" package="R0603" package3d_urn="urn:adsk.eagle:package:23555/2" value="3R3" x="26" y="37.5" smashed="yes" rot="MR180">
+<element name="R2" library="rcl" library_urn="urn:adsk.eagle:library:334" package="R0603" package3d_urn="urn:adsk.eagle:package:23555/2" value="36" x="26" y="37.5" smashed="yes" rot="MR180">
 <attribute name="SPICEPREFIX" value="R" x="26" y="37.5" size="1.778" layer="28" rot="MR180" display="off"/>
 <attribute name="VALUE" x="26" y="38.6354" size="0.8128" layer="26" rot="MR180" align="top-center"/>

Commit message: reverted to old bnc footprint
Parts:
- U$5: value BNC-V -> BNC-VTE-1-1337541-0; device AdapterBoard:TE-5-1634503-1 -> AdapterBoard:BNC-V
Connections:
- net V+: now also U$5.CONDUCTOR1; no longer U$5.C
- net V-: now also U$5.CONDUCTOR2, U$5.SHIELD1, U$5.SHIELD2; no longer U$5.S1, U$5.S2, U$5.S3, U$5.S4
Routing:
- net V-: track 72.0 -> 59.4 mm
- net V+: track 25.8 -> 29.1 mm
- net N$2: track 2.19 -> 1.69 mm
Changed lines of the file:
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@@
 <element name="U$3" library="AdapterBoard" library_urn="urn:adsk.eagle:library:6658125" package="6MM-TERMINAL-POST-BLACK" package3d_urn="urn:adsk.eagle:package:6717096/2" value="6MM-BANANA-PLUGSCREW-BLACK" x="45" y="15.5" smashed="yes" rot="R180"/>
 <element name="U$4" library="AdapterBoard" library_urn="urn:adsk.eagle:library:6658125" package="6MM-TERMINAL-POST-RED" package3d_urn="urn:adsk.eagle:package:6717381/2" value="6MM-BANANA-PLUGSCREW-RED" x="64" y="15.5" smashed="yes" rot="R180"/>
-<element name="U$5" library="AdapterBoard" library_urn="urn:adsk.eagle:library:6658125" package="TE-5-1634503-1" package3d_urn="urn:adsk.eagle:package:7174046/2" value="BNC-V" x="27.5" y="25" smashed="yes" rot="R90"/>
+<element name="U$5" library="AdapterBoard" library_urn="urn:adsk.eagle:library:6658125" package="BNC-V" package3d_urn="urn:adsk.eagle:package:6658128/5" value="BNC-VTE-1-1337541-0" x="27.5" y="25" smashed="yes" rot="R90">
+<attribute name="MANUFACTURERNUMBER" value="TE-Connectivity 1-1337541-0" x="27.5" y="25" size="1.778" layer="27" rot="R90" display="off"/>
+</element>
 <element name="U$6" library="AdapterBoard" library_urn="urn:adsk.eagle:library:6658125" package="1X06_LOCK" package3d_urn="urn:adsk.eagle:package:7198025/2" value="PINHEADER-1X6MALE_LOCK" x="20.15" y="4" smashed="yes"/>
 <element name="U$7" library="AdapterBoard" library_urn="urn:adsk.eagle:library:6658125" package="1X06_LOCK" package3d_urn="urn:adsk.eagle:package:7198025/2" value="PINHEADER-1X6MALE_LOCK" x="20.15" y="46" smashed="yes"/>
@@
 <contactref element="T1" pad="B"/>
 <contactref element="R1" pad="2"/>
-<wire x1="30.35" y1="37.5" x2="30.35" y2="37" width="0.1524" layer="16"/>
 <wire x1="30.35" y1="37.5" x2="31.05" y2="36.8" width="0.1524" layer="16"/>
 <wire x1="31.05" y1="36.8" x2="31.05" y2="36.1" width="0.1524" layer="16"/>
@@
 <signal name="V+">
 <contactref element="U$2" pad="P$1"/>
-<contactref element="U$5" pad="C"/>
+<contactref element="U$5" pad="CONDUCTOR1"/>
 <contactref element="U$4" pad="P$1"/>
 <contactref element="U$7" pad="1"/>
@@
 <wire x1="13.7" y1="16.2" x2="12" y2="14.5" width="1.27" layer="16"/>
 <wire x1="12" y1="14" x2="12" y2="14.5" width="1.27" layer="16"/>
-<wire x1="27.5" y1="25" x2="27.5" y2="27.5" width="0.8128" layer="16"/>
-<wire x1="27.5" y1="27.5" x2="27.94" y2="27.94" width="0.8128" layer="16"/>
 <wire x1="32.95" y1="36.1" x2="32.95" y2="40.646" width="0.1524" layer="16"/>
 <wire x1="32.95" y1="40.646" x2="32.85" y2="40.746" width="0.1524" layer="16"/>
-<wire x1="27.5" y1="25" x2="27.5" y2="26.23" width="0.8128" layer="1"/>
-<wire x1="27.5" y1="26.23" x2="27.94" y2="26.67" width="0.8128" layer="1"/>
-<wire x1="27.5" y1="25" x2="27.5" y2="28.77" width="0.8128" layer="1"/>
-<wire x1="27.5" y1="28.77" x2="27.94" y2="29.21" width="0.8128" layer="1"/>
+<wire x1="27.5" y1="25" x2="27.5" y2="37.66" width="0.8128" layer="1"/>
 </signal>
 <signal name="V-">
@@
 <contactref element="U$8" pad="1"/>
 <contactref element="U$1" pad="P$1"/>
-<contactref element="U$5" pad="S2"/>
-<contactref element="U$5" pad="S3"/>
+<contactref element="U$5" pad="SHIELD1" route="any" routetag="G$1.S"/>
+<contactref element="U$5" pad="SHIELD2" route="any" routetag="G$1.S"/>
 <contactref element="U$3" pad="P$1"/>
 <contactref element="U$6" pad="1"/>
@@
 <wire x1="20" y1="34.5" x2="18" y2="36.5" width="0.1524" layer="16"/>
 <wire x1="18" y1="36.5" x2="6.09" y2="36.5" width="0.1524" layer="16"/>
-<contactref element="U$5" pad="S1"/>
-<contactref element="U$5" pad="S4"/>
-<wire x1="30.63" y1="28.13" x2="30.63" y2="21.87" width="0.8128" layer="16"/>
-<wire x1="24.37" y1="28.13" x2="24.37" y2="21.87" width="0.8128" layer="16"/>
+<contactref element="U$5" pad="CONDUCTOR2" route="any" routetag="G$1.S"/>
 </signal>
 </signals>
