File: Board/Board.brd (EAGLE design)
At the start: 72 x 50 mm, 24 parts, among them IC1 LM334, T1 BC807

Commit message: updated constant current source for power LED
Parts:
- removed R1: 100, rcl:R0603
- removed T1: BC807, DC_LOAD_AU:SOT23-BEC
Connections:
- removed net N$3: IC1.3, R1.1
- removed net N$4: POWER.A, T1.C
- net N$1: no longer POWER.K
- net N$2: now also IC1.3, POWER.K; no longer R1.2, T1.B
- net V+: now also POWER.A; no longer T1.E
Routing:
- net N$4: track 18.5 -> 0.00 mm
- net N$2: track 1.69 -> 13.8 mm
- net N$1: track 13.5 -> 1.91 mm
- net N$3: track 2.11 -> 0.00 mm
- net V+: track 29.1 -> 27.6 mm
Changed lines of the file:
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@@
 <drawing>
 <settings>
-<setting alwaysvectorfont="yes"/>
+<setting alwaysvectorfont="no"/>
 <setting verticaltext="up"/>
 </settings>
-<grid distance="1" unitdist="mm" unit="mm" style="lines" multiple="1" display="yes" altdistance="0.125" altunitdist="mm" altunit="mm"/>
+<grid distance="1" unitdist="mm" unit="mm" style="lines" multiple="1" display="yes" altdistance="0.5" altunitdist="mm" altunit="mm"/>
 <layers>
 <layer number="1" name="Top" color="4" fill="1" visible="yes" active="yes"/>
@@
 <layer number="14" name="Route14" color="22" fill="1" visible="no" active="no"/>
 <layer number="15" name="Route15" color="23" fill="1" visible="no" active="no"/>
-<layer number="16" name="Bottom" color="1" fill="1" visible="no" active="yes"/>
+<layer number="16" name="Bottom" color="1" fill="1" visible="yes" active="yes"/>
 <layer number="17" name="Pads" color="2" fill="1" visible="yes" active="yes"/>
 <layer number="18" name="Vias" color="2" fill="1" visible="yes" active="yes"/>
@@
 <layer number="20" name="Dimension" color="24" fill="1" visible="yes" active="yes"/>
 <layer number="21" name="tPlace" color="7" fill="1" visible="yes" active="yes"/>
-<layer number="22" name="bPlace" color="7" fill="1" visible="no" active="yes"/>
+<layer number="22" name="bPlace" color="7" fill="1" visible="yes" active="yes"/>
 <layer number="23" name="tOrigins" color="15" fill="1" visible="yes" active="yes"/>
-<layer number="24" name="bOrigins" color="15" fill="1" visible="no" active="yes"/>
+<layer number="24" name="bOrigins" color="15" fill="1" visible="yes" active="yes"/>
 <layer number="25" name="tNames" color="7" fill="1" visible="yes" active="yes"/>
-<layer number="26" name="bNames" color="7" fill="1" visible="no" active="yes"/>
+<layer number="26" name="bNames" color="7" fill="1" visible="yes" active="yes"/>
 <layer number="27" name="tValues" color="7" fill="1" visible="no" active="yes"/>
 <layer number="28" name="bValues" color="7" fill="1" visible="no" active="yes"/>
@@
 <layer number="37" name="tTest" color="7" fill="1" visible="no" active="yes"/>
 <layer number="38" name="bTest" color="7" fill="1" visible="no" active="yes"/>
-<layer number="39" name="tKeepout" color="4" fill="11" visible="no" active="yes"/>
-<layer number="40" name="bKeepout" color="1" fill="11" visible="no" active="yes"/>
-<layer number="41" name="tRestrict" color="4" fill="10" visible="no" active="yes"/>
-<layer number="42" name="bRestrict" color="1" fill="10" visible="no" active="yes"/>
+<layer number="39" name="tKeepout" color="4" fill="11" visible="yes" active="yes"/>
+<layer number="40" name="bKeepout" color="1" fill="11" visible="yes" active="yes"/>
+<layer number="41" name="tRestrict" color="4" fill="10" visible="yes" active="yes"/>
+<layer number="42" name="bRestrict" color="1" fill="10" visible="yes" active="yes"/>
 <layer number="43" name="vRestrict" color="2" fill="10" visible="no" active="yes"/>
 <layer number="44" name="Drills" color="7" fill="1" visible="no" active="yes"/>
@@
 <layer number="49" name="Reference" color="7" fill="1" visible="no" active="yes"/>
 <layer number="50" name="dxf" color="7" fill="1" visible="no" active="no"/>
-<layer number="51" name="tDocu" color="7" fill="1" visible="no" active="yes"/>
-<layer number="52" name="bDocu" color="7" fill="1" visible="no" active="yes"/>
+<layer number="51" name="tDocu" color="7" fill="1" visible="yes" active="yes"/>
+<layer number="52" name="bDocu" color="7" fill="1" visible="yes" active="yes"/>
 <layer number="53" name="tGND_GNDA" color="7" fill="9" visible="no" active="no"/>
 <layer number="54" name="bGND_GNDA" color="1" fill="9" visible="no" active="no"/>
@@
 <attribute name="VALUE" x="19.2004" y="33.1966" size="1.27" layer="27" ratio="10"/>
 </element>
-<element name="T1" library="DC_LOAD_AU" library_urn="urn:adsk.eagle:library:220454" package="SOT23-BEC" package3d_urn="urn:adsk.eagle:package:220536/2" value="BC807" x="32" y="35" smashed="yes" rot="MR180">
-<attribute name="VALUE" x="32" y="32.427" size="0.8128" layer="26" rot="MR180" align="center"/>
-</element>
-<element name="R1" library="rcl" library_urn="urn:adsk.eagle:library:334" package="R0603" package3d_urn="urn:adsk.eagle:package:23555/2" value="100" x="29.5" y="37.5" smashed="yes" rot="MR180">
-<attribute name="SPICEPREFIX" value="R" x="29.5" y="37.5" size="1.778" layer="28" rot="MR180" display="off"/>
-<attribute name="VALUE" x="29.499996875" y="38.6354" size="0.8128" layer="26" rot="MR180" align="top-center"/>
-</element>
 <element name="R2" library="rcl" library_urn="urn:adsk.eagle:library:334" package="R0603" package3d_urn="urn:adsk.eagle:package:23555/2" value="36" x="26" y="37.5" smashed="yes" rot="MR180">
 <attribute name="SPICEPREFIX" value="R" x="26" y="37.5" size="1.778" layer="28" rot="MR180" display="off"/>
@@
 </elements>
 <signals>
-<signal name="N$2">
-<contactref element="T1" pad="B"/>
-<contactref element="R1" pad="2"/>
-<wire x1="30.35" y1="37.5" x2="31.05" y2="36.8" width="0.1524" layer="16"/>
-<wire x1="31.05" y1="36.8" x2="31.05" y2="36.1" width="0.1524" layer="16"/>
-</signal>
-<signal name="N$3">
-<contactref element="R1" pad="1"/>
-<contactref element="IC1" pad="3"/>
-<wire x1="28.135" y1="35.6" x2="28.135" y2="36.635" width="0.1524" layer="16"/>
-<wire x1="28.135" y1="36.635" x2="28.65" y2="37.15" width="0.1524" layer="16"/>
-<wire x1="28.65" y1="37.5" x2="28.65" y2="37.15" width="0.1524" layer="16"/>
-</signal>
 <signal name="N$1">
 <contactref element="R2" pad="2"/>
-<contactref element="POWER" pad="K"/>
 <contactref element="IC1" pad="2"/>
 <wire x1="26.865" y1="35.6" x2="26.865" y2="37.485" width="0.1524" layer="16"/>
 <wire x1="26.865" y1="37.485" x2="26.85" y2="37.5" width="0.1524" layer="16"/>
-<wire x1="26.865" y1="35.6" x2="26.865" y2="34.365" width="0.1524" layer="16"/>
-<wire x1="26.865" y1="34.365" x2="26.25" y2="33.75" width="0.1524" layer="16"/>
-<wire x1="26.25" y1="33.75" x2="18.52" y2="33.75" width="0.1524" layer="16"/>
-<wire x1="18.52" y1="33.75" x2="17.27" y2="35" width="0.1524" layer="16"/>
-</signal>
-<signal name="N$4">
-<contactref element="T1" pad="C"/>
-<contactref element="POWER" pad="A"/>
-<wire x1="16.73" y1="33" x2="14.73" y2="35" width="0.1524" layer="16"/>
-<wire x1="32" y1="33.9" x2="30.48" y2="33.9" width="0.1524" layer="16"/>
-<wire x1="30.48" y1="33.9" x2="29.58" y2="33" width="0.1524" layer="16"/>
-<wire x1="29.58" y1="33" x2="16.73" y2="33" width="0.1524" layer="16"/>
 </signal>
 <signal name="V+">
@@
 <contactref element="U$19" pad="P$1"/>
 <contactref element="U$19" pad="P$2"/>
-<contactref element="T1" pad="E"/>
 <polygon width="0.8" layer="1" isolate="0.8128" rank="2">
 <vertex x="0" y="25.875"/>
@@
 <wire x1="13.7" y1="16.2" x2="12" y2="14.5" width="1.27" layer="16"/>
 <wire x1="12" y1="14" x2="12" y2="14.5" width="1.27" layer="16"/>
-<wire x1="32.95" y1="36.1" x2="32.95" y2="40.646" width="0.1524" layer="16"/>
-<wire x1="32.95" y1="40.646" x2="32.85" y2="40.746" width="0.1524" layer="16"/>
-<wire x1="27.5" y1="25" x2="27.5" y2="37.66" width="0.8128" layer="1"/>
+<contactref element="POWER" pad="A"/>
+<wire x1="27.5" y1="25" x2="27.5" y2="40.476" width="1.27" layer="1"/>
+<wire x1="27.5" y1="40.476" x2="27.77" y2="40.746" width="1.27" layer="1"/>
 </signal>
 <signal name="V-">
@@
 <contactref element="U$5" pad="CONDUCTOR2" route="any" routetag="G$1.S"/>
 </signal>
+<signal name="N$2">
+<contactref element="IC1" pad="3"/>
+<contactref element="POWER" pad="K"/>
+<wire x1="28.135" y1="35.6" x2="28.135" y2="34.135" width="0.1524" layer="16"/>
+<wire x1="28.135" y1="34.135" x2="27" y2="33" width="0.1524" layer="16"/>
+<wire x1="27" y1="33" x2="19" y2="33" width="0.1524" layer="16"/>
+<wire x1="19" y1="33" x2="17.27" y2="34.73" width="0.1524" layer="16"/>
+<wire x1="17.27" y1="34.73" x2="17.27" y2="35" width="0.1524" layer="16"/>
+</signal>
 </signals>
